Commit message: feature: add **passive joint** to imitate rubber deform

File: urdf/umi_gripper/umi_gripper.urdf (robot description, URDF)
Before this commit: robot umi_gripper, 22 links, 21 joints
Joints:
- joint left_finger_passive_joint: axis (none) -> 0 1 0; limit (none) -> lower=0 upper=0.01 effort=10 velocity=0.1; type fixed -> prismatic
- joint right_finger_passive_joint: axis (none) -> 0 -1 0; limit (none) -> lower=0 upper=0.01 effort=10 velocity=0.1; mimic (none) -> joint=left_finger_passive_joint multiplier=1 offset=0; type fixed -> prismatic
