Commit message: fixbug: A2-ARM edit finger link initial position

File: urdf/a2-vx300s/a2-vx300s.urdf (robot description, URDF)
Before this commit: robot a2_vx300s, 30 links, 29 joints
Joints:
- joint left_finger_joint: limit lower=0.021 upper=0.057 effort=5 velocity=1 -> lower=0 upper=0.036 effort=5 velocity=1; origin xyz=0 0 0 rpy=0 0 0 -> xyz=0 0.021 0 rpy=0 0 0
- joint right_finger_joint: limit lower=0.021 upper=0.057 effort=5 velocity=1 -> lower=0 upper=0.036 effort=5 velocity=1; origin xyz=0 0 0 rpy=0 0 0 -> xyz=0 -0.021 0 rpy=0 0 0

Commit message: fixbug: A2-ARM edit finger link origin position

File: urdf/a2-vx300s/a2-vx300s.urdf (robot description, URDF)
Before this commit: robot a2_vx300s, 30 links, 29 joints
Joints:
- joint left_finger_joint: origin xyz=0 0.021 0 rpy=0 0 0 -> xyz=0 0.0085 0 rpy=0 0 0
- joint right_finger_joint: origin xyz=0 -0.021 0 rpy=0 0 0 -> xyz=0 -0.0085 0 rpy=0 0 0

Commit message: perf: A2-ARM edit collision mesh

File: urdf/a2-vx300s/a2-vx300s.urdf (robot description, URDF)
Before this commit: robot a2_vx300s, 30 links, 29 joints
Links:
- link vx300s_base_link: geometry collision box size=0.115 0.082 0.045; collision cylinder length=0.067 radius=0.069
- link vx300s_gripper_bar_link: geometry visual mesh filename=meshes/vx300s_9_gripper_bar.stl scale=0.001 0.001 0.001
- link vx300s_gripper_link: geometry collision box size=0.0447 0.150 0.046; visual mesh filename=meshes/vx300s_7_gripper.stl scale=0.001 0.001 0.001
- link vx300s_left_finger_link: geometry collision box size=0.06 0.0205 0.061; visual mesh filename=meshes/vx300s_10_gripper_finger.stl scale=0.001 0.001 0.001
- link vx300s_lower_forearm_link: geometry collision box size=0.118 0.1 0.0395; visual mesh filename=meshes/vx300s_5_lower_forearm.stl scale=0.001 0.001 0.001
- link vx300s_right_finger_link: geometry collision box size=0.06 0.0205 0.061; visual mesh filename=meshes/vx300s_10_gripper_finger.stl scale=0.001 0.001 0.001
- link vx300s_shoulder_link: geometry collision box size=0.0335 0.102 0.0585; visual mesh filename=meshes/vx300s_2_shoulder.stl scale=0.001 0.001 0.001
- link vx300s_upper_arm_link: geometry collision box size=0.020 0.040 0.295; collision box size=0.06375 0.1012 0.0419
- link vx300s_upper_forearm_link: geometry collision box size=0.166791 0.0452 0.0315; visual mesh filename=meshes/vx300s_4_upper_forearm.stl scale=0.001 0.001 0.001
- link vx300s_wrist_link: geometry collision box size=0.034 0.055 0.0465; visual mesh filename=meshes/vx300s_6_wrist.stl scale=0.001 0.001 0.001

Commit message: perf: separate holder and finger joint (for rubber passive joint)

File: urdf/a2-vx300s/a2-vx300s.urdf (robot description, URDF)
Before this commit: robot a2_vx300s, 31 links, 30 joints
Links:
- added link vx300s_left_carriage, mass 0.020; visual mesh filename=meshes/umi_left_finger_holder.stl scale=1 1 1
- added link vx300s_right_carriage, mass 0.020; visual mesh filename=meshes/umi_right_finger_holder.stl scale=1 1 1
Joints:
- added joint left_finger_passive_joint: type prismatic, parent vx300s_left_carriage, child vx300s_left_finger_link, origin xyz=0 0 0 rpy=0 0 0, axis 0 1 0, limit lower=0 upper=0.01 effort=10 velocity=0.1
- added joint right_finger_passive_joint: type prismatic, parent vx300s_right_carriage, child vx300s_right_finger_link, origin xyz=0 0 0 rpy=0 0 0, axis 0 -1 0, limit lower=0 upper=0.01 effort=10 velocity=0.1, mimic joint=left_finger_passive_joint multiplier=1 offset=0
- joint left_finger_joint: child vx300s_left_finger_link -> vx300s_left_carriage
- joint right_finger_joint: child vx300s_right_finger_link -> vx300s_right_carriage

Commit message: perf: add top cover

File: urdf/a2-vx300s/a2-vx300s.urdf (robot description, URDF)
Before this commit: robot a2_vx300s, 33 links, 32 joints
Links:
- added link umi_base_top, mass 0.050; visual mesh filename=meshes/umi_base_top.stl scale=1 1 1
- link vx300s_gripper_bar_link: geometry 
Joints:
- added joint umi_base_top_joint: type fixed, parent vx300s_fingers_link, child umi_base_top, origin xyz=0.0 0.0 0.0 rpy=0 0 0, axis 0 1 0

Commit message: perf: add black tape

File: urdf/a2-vx300s/a2-vx300s.urdf (robot description, URDF)
Before this commit: robot a2_vx300s, 37 links, 36 joints
Links:
- added link left_tape, mass 0.005; visual box size=0.12 0.0258 0.00002
- added link right_tape, mass 0.005; visual box size=0.12 0.0258 0.00002
Joints:
- added joint fix_left_tape_and_left_finger: type fixed, parent vx300s_left_finger_link, child left_tape, origin xyz=0 0 0 rpy=0 0 0
- added joint fix_right_tape_and_right_finger: type fixed, parent vx300s_right_finger_link, child right_tape, origin xyz=0 0 0 rpy=0 0 0
- joint umi_base_bottom_joint: parent vx300s/fingers_link -> vx300s_fingers_link

Commit message: perf: add bottom cover

File: urdf/a2-vx300s/a2-vx300s.urdf (robot description, URDF)
Before this commit: robot a2_vx300s, 36 links, 35 joints
Links:
- added link umi_base_bottom, mass 0.055; visual mesh filename=meshes/umi_base_bottom.stl scale=1 1 1
Joints:
- added joint umi_base_bottom_joint: type fixed, parent vx300s/fingers_link, child umi_base_bottom, origin xyz=0.0 0.0 0.0 rpy=0 0 0, axis 0 1 0

Commit message: perf: add mirror

File: urdf/a2-vx300s/a2-vx300s.urdf (robot description, URDF)
Before this commit: robot a2_vx300s, 34 links, 33 joints
Links:
- added link left_mirror, mass 0.005; visual box size=0.06 0.0374 0.0002
- added link right_mirror, mass 0.005; visual box size=0.06 0.0374 0.0002
Joints:
- added joint fix_linear_rail_and_left_mirror: type fixed, parent umi_base_top, child left_mirror, origin xyz=0 0 0 rpy=0 0 0
- added joint fix_linear_rail_and_right_mirror: type fixed, parent umi_base_top, child right_mirror, origin xyz=0 0 0 rpy=0 0 0
